File: PICDevBoard-V1RevA/PICDevBoard-V1RevA.sch (EAGLE design)
At the start: 15 parts, among them IC1 PIC18F2550, J1 DCJ0202

Commit message: Silk
Adicionado nome dos pinos no silk (top layer)
Connections:
- net GND: now also SV2.7; no longer SV2.10
- net RC0: now also SV2.8; no longer SV2.7
- net RC1: now also SV2.9; no longer SV2.8
- net RC2: now also SV2.10; no longer SV2.9
Changed lines of the file:
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@@
 <?xml version="1.0" encoding="utf-8"?>
 <!DOCTYPE eagle SYSTEM "eagle.dtd">
-<eagle version="6.1">
+<eagle version="6.4">
 <drawing>
 <settings>
@@
 </segment>
 <segment>
-<pinref part="SV2" gate="G$1" pin="10"/>
-<wire x1="71.12" y1="139.7" x2="73.66" y2="139.7" width="0.1524" layer="91"/>
-<label x="73.66" y="139.7" size="1.27" layer="95" font="vector" xref="yes"/>
+<pinref part="SV2" gate="G$1" pin="7"/>
+<wire x1="71.12" y1="147.32" x2="73.66" y2="147.32" width="0.1524" layer="91"/>
+<label x="73.66" y="147.32" size="1.27" layer="95" font="vector" xref="yes"/>
 </segment>
 </net>
@@
 </segment>
 <segment>
-<pinref part="SV2" gate="G$1" pin="7"/>
-<wire x1="71.12" y1="147.32" x2="73.66" y2="147.32" width="0.1524" layer="91"/>
-<label x="73.66" y="147.32" size="1.27" layer="95" font="vector" xref="yes"/>
+<pinref part="SV2" gate="G$1" pin="8"/>
+<wire x1="71.12" y1="144.78" x2="73.66" y2="144.78" width="0.1524" layer="91"/>
+<label x="73.66" y="144.78" size="1.27" layer="95" font="vector" xref="yes"/>
 </segment>
 </net>
@@
 </segment>
 <segment>
-<pinref part="SV2" gate="G$1" pin="8"/>
-<wire x1="71.12" y1="144.78" x2="73.66" y2="144.78" width="0.1524" layer="91"/>
-<label x="73.66" y="144.78" size="1.27" layer="95" font="vector" xref="yes"/>
+<pinref part="SV2" gate="G$1" pin="9"/>
+<wire x1="71.12" y1="142.24" x2="73.66" y2="142.24" width="0.1524" layer="91"/>
+<label x="73.66" y="142.24" size="1.27" layer="95" font="vector" xref="yes"/>
 </segment>
 </net>
@@
 </segment>
 <segment>
-<pinref part="SV2" gate="G$1" pin="9"/>
-<wire x1="71.12" y1="142.24" x2="73.66" y2="142.24" width="0.1524" layer="91"/>
-<label x="73.66" y="142.24" size="1.27" layer="95" font="vector" xref="yes"/>
-</segment>
-</net>
+<pinref part="SV2" gate="G$1" pin="10"/>
+<wire x1="71.12" y1="139.7" x2="73.66" y2="139.7" width="0.1524" layer="91"/>
+<label x="73.66" y="139.7" size="1.27" layer="95" font="vector" xref="yes"/>
+</segment>
+</net>

Commit message: Routing
Continuação do roteamento
Parts:
- added SV4, SV5: (no value), con-lstb:MA03-1
Connections:
- net 5VICSP: now also SV1.2; no longer SV1.6
- net 5VUSB: now also SV1.6; no longer SV1.2
- net GND: now also SV5.1, SV5.2, SV5.3, USB1.GND@1, USB1.GND@2, USB1.GND@3, USB1.GND@4
- net VCC: now also SV4.1, SV4.2, SV4.3
Other:
- note added: "Adicionar capacitor entre HIPWR"
- note removed: "Pontos GND HI-POWER"
- note removed: "Pontos VCC HI-POWER"
Changed lines of the file:
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@@
 <part name="SV2" library="con-lsta" deviceset="FE10-1" device=""/>
 <part name="SV3" library="con-lsta" deviceset="FE10-1" device=""/>
+<part name="GND8" library="supply1" deviceset="GND" device=""/>
+<part name="GND9" library="supply1" deviceset="GND" device=""/>
+<part name="SV4" library="con-lstb" deviceset="MA03-1" device=""/>
+<part name="SV5" library="con-lstb" deviceset="MA03-1" device=""/>
+<part name="GND10" library="supply1" deviceset="GND" device=""/>
+<part name="P+6" library="supply1" deviceset="VCC" device=""/>
+<part name="GND11" library="supply1" deviceset="GND" device=""/>
+<part name="GND12" library="supply1" deviceset="GND" device=""/>
 </parts>
 <sheets>
@@
 <text x="5.588" y="68.58" size="1.778" layer="94" font="vector" ratio="11">5V DC JACK @ 1A</text>
 <wire x1="5.08" y1="48.26" x2="45.72" y2="48.26" width="0.1524" layer="94" style="dashdot"/>
-<wire x1="45.72" y1="48.26" x2="45.72" y2="15.24" width="0.1524" layer="94" style="dashdot"/>
-<wire x1="45.72" y1="15.24" x2="5.08" y2="15.24" width="0.1524" layer="94" style="dashdot"/>
-<wire x1="5.08" y1="15.24" x2="5.08" y2="48.26" width="0.1524" layer="94" style="dashdot"/>
+<wire x1="45.72" y1="48.26" x2="45.72" y2="7.62" width="0.1524" layer="94" style="dashdot"/>
+<wire x1="45.72" y1="7.62" x2="5.08" y2="7.62" width="0.1524" layer="94" style="dashdot"/>
+<wire x1="5.08" y1="7.62" x2="5.08" y2="48.26" width="0.1524" layer="94" style="dashdot"/>
 <text x="5.842" y="45.72" size="1.778" layer="94" font="vector" ratio="11">USB</text>
 <wire x1="5.08" y1="172.72" x2="45.72" y2="172.72" width="0.1524" layer="94" style="dashdot"/>
@@
 <text x="147.32" y="157.48" size="1.778" layer="94" font="vector">Pontos de GND</text>
 <text x="147.32" y="154.94" size="1.778" layer="94" font="vector">Pontos de VCC</text>
-<text x="147.32" y="152.4" size="1.778" layer="94" font="vector">Pontos GND HI-POWER</text>
-<text x="147.32" y="149.86" size="1.778" layer="94" font="vector">Pontos VCC HI-POWER</text>
-<text x="147.32" y="147.32" size="1.778" layer="94" font="vector">Filtro PI</text>
-<text x="147.32" y="144.78" size="1.778" layer="94" font="vector">On/Off Switch</text>
-<text x="147.32" y="142.24" size="1.778" layer="94" font="vector">Reset</text>
+<text x="147.32" y="144.78" size="1.778" layer="94" font="vector">Filtro PI</text>
+<text x="147.32" y="152.4" size="1.778" layer="94" font="vector">On/Off Switch</text>
+<text x="147.32" y="149.86" size="1.778" layer="94" font="vector">Reset</text>
+<text x="147.32" y="147.32" size="1.778" layer="94" font="vector">Adicionar capacitor entre HIPWR</text>
 </plain>
 <instances>
@@
 <instance part="GND7" gate="1" x="27.94" y="63.5" rot="R90"/>
 <instance part="P+5" gate="VCC" x="35.56" y="58.42" rot="R270"/>
-<instance part="USB1" gate="G$1" x="17.78" y="30.48"/>
-<instance part="GND5" gate="1" x="33.02" y="20.32"/>
-<instance part="P+3" gate="VCC" x="33.02" y="40.64"/>
+<instance part="USB1" gate="G$1" x="17.78" y="27.94"/>
+<instance part="GND5" gate="1" x="33.02" y="17.78"/>
+<instance part="P+3" gate="VCC" x="33.02" y="38.1"/>
 <instance part="SV2" gate="G$1" x="63.5" y="152.4" rot="MR180"/>
 <instance part="SV3" gate="G$1" x="63.5" y="116.84" rot="MR180"/>
+<instance part="GND8" gate="1" x="22.86" y="12.7"/>
+<instance part="GND9" gate="1" x="10.16" y="40.64" rot="R180"/>
+<instance part="SV4" gate="G$1" x="63.5" y="83.82"/>
+<instance part="SV5" gate="G$1" x="63.5" y="60.96"/>
+<instance part="GND10" gate="1" x="76.2" y="53.34"/>
+<instance part="P+6" gate="VCC" x="76.2" y="93.98"/>
+<instance part="GND11" gate="1" x="10.16" y="12.7"/>
+<instance part="GND12" gate="1" x="22.86" y="40.64" rot="R180"/>
 </instances>
 <busses>
@@
 <pinref part="USB1" gate="G$1" pin="GND"/>
 <pinref part="GND5" gate="1" pin="GND"/>
-<wire x1="30.48" y1="25.4" x2="33.02" y2="25.4" width="0.1524" layer="91"/>
-<wire x1="33.02" y1="25.4" x2="33.02" y2="22.86" width="0.1524" layer="91"/>
+<wire x1="30.48" y1="22.86" x2="33.02" y2="22.86" width="0.1524" layer="91"/>
+<wire x1="33.02" y1="22.86" x2="33.02" y2="20.32" width="0.1524" layer="91"/>
+</segment>
+<segment>
+<pinref part="USB1" gate="G$1" pin="GND@4"/>
+<pinref part="GND8" gate="1" pin="GND"/>
+<wire x1="22.86" y1="15.24" x2="22.86" y2="17.78" width="0.1524" layer="91"/>
+</segment>
+<segment>
+<pinref part="USB1" gate="G$1" pin="GND@1"/>
+<pinref part="GND9" gate="1" pin="GND"/>
 </segment>
 <segment>
@@
 <wire x1="71.12" y1="147.32" x2="73.66" y2="147.32" width="0.1524" layer="91"/>
 <label x="73.66" y="147.32" size="1.27" layer="95" font="vector" xref="yes"/>
+</segment>
+<segment>
+<pinref part="SV5" gate="G$1" pin="1"/>
+<pinref part="GND10" gate="1" pin="GND"/>
+<wire x1="71.12" y1="58.42" x2="76.2" y2="58.42" width="0.1524" layer="91"/>
+<wire x1="76.2" y1="58.42" x2="76.2" y2="55.88" width="0.1524" layer="91"/>
+<pinref part="SV5" gate="G$1" pin="2"/>
+<wire x1="71.12" y1="60.96" x2="76.2" y2="60.96" width="0.1524" layer="91"/>
+<wire x1="76.2" y1="60.96" x2="76.2" y2="58.42" width="0.1524" layer="91"/>
+<junction x="76.2" y="58.42"/>
+<pinref part="SV5" gate="G$1" pin="3"/>
+<wire x1="71.12" y1="63.5" x2="76.2" y2="63.5" width="0.1524" layer="91"/>
+<wire x1="76.2" y1="63.5" x2="76.2" y2="60.96" width="0.1524" layer="91"/>
+<junction x="76.2" y="60.96"/>
+</segment>
+<segment>
+<pinref part="USB1" gate="G$1" pin="GND@3"/>
+<pinref part="GND11" gate="1" pin="GND"/>
+<wire x1="10.16" y1="15.24" x2="10.16" y2="17.78" width="0.1524" layer="91"/>
+</segment>
+<segment>
+<pinref part="USB1" gate="G$1" pin="GND@2"/>
+<pinref part="GND12" gate="1" pin="GND"/>
 </segment>
 </net>
@@
 <pinref part="P+4" gate="VCC" pin="VCC"/>
 </segment>
+<segment>
+<pinref part="SV4" gate="G$1" pin="1"/>
+<pinref part="P+6" gate="VCC" pin="VCC"/>
+<wire x1="71.12" y1="81.28" x2="76.2" y2="81.28" width="0.1524" layer="91"/>
+<wire x1="76.2" y1="81.28" x2="76.2" y2="83.82" width="0.1524" layer="91"/>
+<pinref part="SV4" gate="G$1" pin="3"/>
+<wire x1="76.2" y1="83.82" x2="76.2" y2="86.36" width="0.1524" layer="91"/>
+<wire x1="76.2" y1="86.36" x2="76.2" y2="91.44" width="0.1524" layer="91"/>
+<wire x1="71.12" y1="86.36" x2="76.2" y2="86.36" width="0.1524" layer="91"/>
+<junction x="76.2" y="86.36"/>
+<pinref part="SV4" gate="G$1" pin="2"/>
+<wire x1="71.12" y1="83.82" x2="76.2" y2="83.82" width="0.1524" layer="91"/>
+<junction x="76.2" y="83.82"/>
+</segment>
 </net>
 <net name="VPP" class="0">
@@
 <segment>
 <pinref part="USB1" gate="G$1" pin="D+"/>
-<wire x1="30.48" y1="30.48" x2="33.02" y2="30.48" width="0.1524" layer="91"/>
-<label x="33.02" y="30.48" size="1.27" layer="95" font="vector" xref="yes"/>
+<wire x1="30.48" y1="27.94" x2="33.02" y2="27.94" width="0.1524" layer="91"/>
+<label x="33.02" y="27.94" size="1.27" layer="95" font="vector" xref="yes"/>
 </segment>
 </net>
@@
 <segment>
 <pinref part="USB1" gate="G$1" pin="D-"/>
-<wire x1="30.48" y1="33.02" x2="33.02" y2="33.02" width="0.1524" layer="91"/>
-<label x="33.02" y="33.02" size="1.27" layer="95" font="vector" xref="yes"/>
+<wire x1="30.48" y1="30.48" x2="33.02" y2="30.48" width="0.1524" layer="91"/>
+<label x="33.02" y="30.48" size="1.27" layer="95" font="vector" xref="yes"/>
 </segment>
 </net>
@@
 <net name="5VUSB" class="0">
 <segment>
-<pinref part="SV1" gate="1" pin="2"/>
-<wire x1="22.86" y1="78.74" x2="20.32" y2="78.74" width="0.1524" layer="91"/>
-<label x="20.32" y="78.74" size="1.27" layer="95" font="vector" ratio="11" rot="R180" xref="yes"/>
-</segment>
-<segment>
 <pinref part="USB1" gate="G$1" pin="VCC"/>
 <pinref part="P+3" gate="VCC" pin="VCC"/>
-<wire x1="30.48" y1="35.56" x2="33.02" y2="35.56" width="0.1524" layer="91"/>
-<wire x1="33.02" y1="35.56" x2="33.02" y2="38.1" width="0.1524" layer="91"/>
+<wire x1="30.48" y1="33.02" x2="33.02" y2="33.02" width="0.1524" layer="91"/>
+<wire x1="33.02" y1="33.02" x2="33.02" y2="35.56" width="0.1524" layer="91"/>
+</segment>
+<segment>
+<pinref part="SV1" gate="1" pin="6"/>
+<wire x1="22.86" y1="83.82" x2="20.32" y2="83.82" width="0.1524" layer="91"/>
+<label x="20.32" y="83.82" size="1.27" layer="95" font="vector" ratio="11" rot="R180" xref="yes"/>
 </segment>
 </net>
@@
 </segment>
 <segment>
-<pinref part="SV1" gate="1" pin="6"/>
-<wire x1="22.86" y1="83.82" x2="20.32" y2="83.82" width="0.1524" layer="91"/>
-<label x="20.32" y="83.82" size="1.27" layer="95" font="vector" ratio="11" rot="R180" xref="yes"/>
-</segment>
-</net>
+<pinref part="SV1" gate="1" pin="2"/>
+<wire x1="22.86" y1="78.74" x2="20.32" y2="78.74" width="0.1524" layer="91"/>
+<label x="20.32" y="78.74" size="1.27" layer="95" font="vector" ratio="11" rot="R180" xref="yes"/>
+</segment>
+</net>

Commit message: Routing
Parts:
- added C5: 10u, rcl:C-EUC0805
Connections:
- net 5VJACK: now also J1.1; no longer J1.2, J1.3
- net GND: now also C5.2, J1.3; no longer J1.1
- net VCC: now also C5.1
Other:
- note added: "GPIO"
- note added: "HI-POWER"
- note added: "Iuri Castro"
- note removed: "Adicionar capacitor entre HIPWR"
- note removed: "Filtro PI"
- note removed: "On/Off Switch"
- note removed: "Pontos de GND"
- note removed: "Pontos de VCC"
- note removed: "Reset"
- moved on the sheet: C3, C4, IC1, R1, R2, R3, SV1, SV2, SV3, SV4, SV5
