File: IronDriverInterfaceRevA/IronDriverInterfaceRevA.sch (EAGLE design)
At the start: 31 parts, among them IC1 PIC18F2550, IC2 TL074P, IC3 7805TV, IC4 TL072P, Q1 BC557C

Commit message: Routing IronDriver
Parts:
- removed 24VRMS, HEATER: (no value), con-ptr500:AK500/2
- removed D1, D2, D3, D4: 1N4004, diode:1N4004
- removed FUSE1: (no value), FUSEHOLDER:FUSEHOLDER
- removed IC1: PIC18F2550, PIC18F2550:PIC18F2550
- removed IC2: TL074P, linear:TL074P
- removed IC3: 7805TV, linear:7805TV
- removed IC4: TL072P, linear:TL072P
- removed ICSP: (no value), con-lstb:MA04-1
- removed J1: (no value), FFC:FFC14X1
- removed MOC1: MOC3011M, optocoupler:MOC3011M
- removed OPTO1, OPTO2: 4N25M, optocoupler:4N25M
- removed PTC: (no value), con-ptr500:AK500/3
- removed Q1: BC557C, transistor-pnp:BC557C
- removed R10, R11, R7, R8, R9: (no value), rcl:R-EU_0207/7
- removed TRIAC1: BTA16, BTA16-600BRG:BTA16-600BRG
- added C2, C3: (no value), rcl:C-EUC0805
- added ENC1: (no value), IronDriverLibrary:ENCODER
- added LCD1: (no value), IronDriverLibrary:HC0821
- added SV1: (no value), con-lstb:MA07-2
- added T1: (no value), transistor:MMBT3904LT1-NPN-SOT23-BEC
- C1: value 100nF -> (none)
- R1, R2: value 1k8 -> (none); device rcl:R-EU_0207/7 -> rcl:R-EU_R0805
- R3, R6: value 10k -> (none)
- R4: value 33R -> (none); device rcl:R-EU_0207/7 -> rcl:R-EU_R0805
- R5: value 470R -> (none); device rcl:R-EU_0207/7 -> rcl:R-EU_R0805
Connections:
- removed net +8V: IC2P.V+, IC4P.V+, R11.1
- removed net +PTC: IC2A.+IN, IC4A.-IN, PTC-1.KL, R11.2
- removed net -PTC: IC2B.+IN, PTC-2.KL, Q1.E
- removed net ADC_IN: IC1.RA0/AN0, IC2D.-IN, IC2D.OUT
- removed net HEATER: IC1.RC0/T1OSO/T13CKI, R5.1
- removed net HEATER_LIVE: HEATER-1.KL, R4.2, TRIAC1.A2
- removed net LCD_D4: IC1.RA1/AN1
- removed net LCD_D5: IC1.RA3/AN3/VREF+
- removed net LCD_D6: IC1.RA4/T0CKI/C1OUT/RCV
- removed net LCD_D7: IC1.RA5/AN4/!SS!/HLVDIN/C2OUT
- removed net LIVE: D1.A, D3.C, FUSE1.P$2, R1.1, TRIAC1.A1
- removed net N$10: MOC1.A1, R4.1
- removed net N$11: 24VRMS-2.KL, FUSE1.P$1
- removed net N$12: IC2B.-IN, IC2B.OUT, R8.1
- removed net N$19: IC2C.OUT, IC2D.+IN, R7.2
- removed net N$21: IC4A.+IN
- removed net N$4: OPTO1.A, OPTO2.C, R1.2
- removed net N$5: IC2C.-IN, R7.1, R8.2
- removed net N$6: IC2C.+IN, R10.1, R9.2
- removed net N$8: MOC1.A2, TRIAC1.G
- removed net N$9: IC2A.-IN, IC2A.OUT, R9.1
- removed net NEUTRAL: 24VRMS-1.KL, D2.C, D4.A, HEATER-2.KL, R2.1
- removed net PGC: IC1.RB6/KBI2/PGC, ICSP.2
- removed net PGD: IC1.RB7/KBI3/PGD, ICSP.3
- removed net VGND: IC1.RA2/AN2/VREF-/CVREF, IC4B.-IN, IC4B.OUT, R10.2
- removed net VPP: IC1.!MCLR!/VPP/RE3, ICSP.4, R6.1
- removed net ZEROCROSSING: IC1.RB0/AN12/INT0/FLT0/SDI/SDA, OPTO1.COL, OPTO2.COL, R3.1
- new net LCD_VO: LCD1.VO
- new net LED: SV1.2
- new net N$17: ENC1.B, R4.1, R6.1
- net ENC_A: now also C3.1, R3.1, SV1.4; no longer IC1.RB1/AN10/INT1/SCK/SCL, J1.4
- net ENC_B: now also C2.1, R4.2, SV1.6; no longer IC1.RB2/AN8/INT2/VMO, J1.6
- net GND: now also C2.2, C3.2, ENC1.COM, LCD1.VSS, SV1.3, SV1.8, T1.E; no longer D2.A, D3.A, IC1.VSS@1, IC1.VSS@2, IC2P.V-, IC4P.V-, ICSP.1, J1.3, J1.8, MOC1.C, OPTO1.EMI, OPTO2.EMI, PTC-3.KL, Q1.C
- net LCD_BL: now also R1.1, SV1.1; no longer J1.1
- net LCD_D0: now also LCD1.DB4, SV1.11; no longer J1.11
- net LCD_D1: now also LCD1.DB5, SV1.13; no longer J1.13
- net LCD_D2: now also LCD1.DB6, SV1.7; no longer J1.7
- net LCD_D3: now also LCD1.DB7, SV1.9; no longer J1.9
- net LCD_E: now also LCD1.E, SV1.14; no longer IC1.RC7/RX/DT/SDO, J1.14
- net LCD_RS: now also LCD1.RS, SV1.10; no longer IC1.RC6/TX/CK, J1.10
- net LCD_RW: now also LCD1.R/W, SV1.12; no longer IC1.RC2/CCP1, J1.12
- net N$1: now also LCD1.LEDK, R2.2; no longer MOC1.A, R5.2
- net N$16: now also ENC1.A, R3.2, R5.1; no longer D1.C, D4.C
- net N$2: now also R2.1, T1.C; no longer IC4A.OUT, Q1.B
- net N$3: now also R1.2, T1.B; no longer OPTO1.C, OPTO2.A, R2.2
- net VCC: now also LCD1.LEDA, LCD1.VDD, R5.2, SV1.5; no longer IC1.VDD, J1.5, R3.2
Other:
- note removed: "+2V"
- note removed: "1N4148"
- note removed: "Acionamento do Heater"
- note removed: "Adicionar LM7805"
- note removed: "Adicionar capacitores de filtro"
- note removed: "Adicionar trimpot 10k ou 100k"
- note removed: "Capacitor de filtro na ordem de 100uF@35V"
- note removed: "Circuito Zerocrossing"
- note removed: "Conector AC 24VRMS"
- note removed: "Conector Heater"
- note removed: "Conector PTC Ferro de Solda"
- note removed: "D1, D2, D3, D4"
- note removed: "Substituir por ponte completa e DCDC"
- note removed: "Virtual Ground"
