File: IronDriverRevA/IronDriverRevA.sch (EAGLE design)
At the start: 33 parts, among them IC1 PIC18F2550, IC2 TL074P, IC3 7805TV, IC4 TL072P, Q1 BC557C

Commit message: Routing
DCDC added
Parts:
- added C2: 100uF @ 35V, rcl:CPOL-EUE2.5-7
- added C3: 200pF, rcl:C-EU025-025X050
- added C4: 25uF, rcl:CPOL-EUE2.5-7
- added C5: 100uF, rcl:CPOL-EUE2-5
- added C6: .1uF @ 5V, rcl:C-EU025-025X050
- added C7: .33uF @ 8V, rcl:C-EU025-025X050
- added D5: 1N5819-T, diode:1N5819-T
- added IC5: MC34063AP, mc34063:MC34063AP
- added L1: 210uH, rcl:L-US6000-XXX-RC
- added L2: 1uH, rcl:L-US6000-XXX-RC
- added R14: 2.4k, rcl:R-EU_0207/7
- added R15: 13k, rcl:R-EU_0207/7
- added R16: 1.5R, rcl:R-EU_0207/7
Connections:
- removed net VCC: C1.1, IC1.VDD, J1.5, R3.2, R6.2
- new net +5V: C1.1, C6.1, IC1.VDD, IC3.VO, J1.5, R3.2, R6.2
- new net N$13: D5.C, IC5.SWE, L1.1
- new net N$14: IC5.FB, R14.2, R15.2
- new net N$15: IC5.DC, IC5.IS, IC5.SWC, R16.2
- new net N$18: C3.1, IC5.TC
- new net N$20: C2.+, D1.C, D4.C, IC5.VCC, R16.1
- net +8V: now also C5.+, C7.1, IC3.VI, L2.2, R15.1
- net GND: now also C2.-, C3.2, C4.-, C5.-, C6.2, C7.2, D5.A, IC3.GND, IC5.GND, R14.1
- net N$16: now also C4.+, L1.2, L2.1; no longer D1.C, D4.C
Other:
- note removed: "Adicionar LM7805"
- note removed: "Adicionar capacitores de filtro"
- note removed: "Capacitor de filtro na ordem de 100uF@35V"
- note removed: "Substituir por ponte completa e DCDC"
- moved on the sheet: D1, D2, D3, D4, IC3, MOC1, R4, R5, TRIAC1
