File: IronDriverRevA/IronDriverRevA.sch (EAGLE design)
At the start: 31 parts, among them IC1 PIC18F2550, IC2 TL074P, IC3 7805TV, IC4 TL072P, Q1 BC557C

Commit message: Routing
Parts:
- added R12, R13: 10k, rcl:R-TRIMM3296W
- R10, R7, R8, R9: value (none) -> 100k
- R11: value (none) -> 220
- R3, R6: device rcl:R-EU_R0805 -> rcl:R-EU_0207/7
Connections:
- new net N$7: IC4B.+IN, R13.S
- net +8V: now also R12.E, R13.E
- net GND: now also R12.A, R13.A
- net N$21: now also R12.S
Other:
- note added: "Casar R9 com R8 e R10 com R7"
- note removed: "Adicionar trimpot 10k ou 100k"
- moved on the sheet: IC4B, Q1, R11

Commit message: Routing
Parts:
- removed D1, D2, D3, D4: 1N4004, diode:1N4004
- added C2: (no value), rcl:C-EUC0805
- added IC5: (no value), LM2596:LM2596
- added IC6: (no value), RS207:RS207
Connections:
- removed net N$16: D1.C, D4.C
- net +8V: now also C2.1
- net GND: now also C2.2, IC5.GND, IC6.-; no longer D2.A, D3.A
- net LIVE: now also IC6.AC2; no longer D1.A, D3.C
- net NEUTRAL: now also IC6.AC1; no longer D2.C, D4.A
Other:
- note removed: "1N4148"
- note removed: "Adicionar LM7805"
- note removed: "D1, D2, D3, D4"
- note removed: "Substituir por ponte completa e DCDC"
- moved on the sheet: IC3, MOC1, R4, R5, TRIAC1

Commit message: Added ChikenControlelr
Parts:
- added JUMPER1: (no value), rcl:R-EU_M1206
Changed lines of the file:
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@@
 <part name="C2" library="rcl" deviceset="C-EU" device="C0805"/>
 <part name="GND16" library="supply1" deviceset="GND" device=""/>
+<part name="JUMPER1" library="rcl" deviceset="R-EU_" device="M1206"/>
 </parts>
 <sheets>
@@
 <instance part="C2" gate="G$1" x="63.5" y="111.76" rot="R90"/>
 <instance part="GND16" gate="1" x="73.66" y="111.76" rot="R90"/>
+<instance part="JUMPER1" gate="G$1" x="38.1" y="25.4"/>
 </instances>
 <busses>
