File: IronDriverRevA/IronDriverRevA.sch (EAGLE design)
At the start: 46 parts, among them IC1 PIC18F2550, IC2 TL074P, IC3 7805TV, IC4 TL072P, IC5 MC34063AP, Q1 BC557C

Commit message: Finalizando Roteamento
Parts:
- added JMP1, JMP2, JMP3, JMP4, JMP5, JMP6, JMP7: (no value), rcl:R-EU_R1206
Connections:
- removed net LCD_D4: IC1.RA1/AN1
- removed net LCD_D5: IC1.RA3/AN3/VREF+
- removed net LCD_D6: IC1.RA4/T0CKI/C1OUT/RCV
- removed net LCD_D7: IC1.RA5/AN4/!SS!/HLVDIN/C2OUT
- new net +5V_JMP4: J1.5, JMP4.1, R6.2
- new net +5V_MC: C1.1, IC1.VDD, JMP3.1
- new net GND_JMP5: J1.3, JMP5.1
- new net N$17: J1.6, JMP1.2
- new net N$23: J1.9, JMP7.2
- new net N$24: JMP6.2, JMP7.1
- new net ZEROCROSSING_B: JMP2.1, OPTO1.COL, OPTO2.COL, R3.1
- net +5V: now also JMP3.2, JMP4.2; no longer C1.1, IC1.VDD, J1.5, R6.2
- net ENC_B: now also JMP1.1; no longer J1.6
- net GND: now also JMP5.2; no longer J1.3
- net LCD_BL: now also IC1.RB4/AN11/KBI0
- net LCD_D0: now also IC1.RC1/T1OSI/CCP2/!UOE
- net LCD_D1: now also IC1.RC6/TX/CK
- net LCD_D2: now also IC1.RA1/AN1
- net LCD_D3: now also IC1.RB5/KBI1/PGM, JMP6.1; no longer J1.9
- net LCD_E: now also IC1.RC2/CCP1; no longer IC1.RC7/RX/DT/SDO
- net LCD_RS: now also IC1.RB3/AN9/CCP2/VPO; no longer IC1.RC6/TX/CK
- net LCD_RW: now also IC1.RC7/RX/DT/SDO; no longer IC1.RC2/CCP1
- net ZEROCROSSING: now also JMP2.2; no longer OPTO1.COL, OPTO2.COL, R3.1
Other:
- note added: "2A @ 35V"
- note added: "Colocar capacitores de bypass"
- note added: "Fonte de Alimentacao"
- note added: "Iuri Castro"
- moved on the sheet: 24VRMS-1, 24VRMS-2, C2, C3, C4, C5, C6, C7, D1, D2, D3, D4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

Commit message: Ajustes de trilhas
Parts:
- L2: device rcl:L-US6000-XXX-RC -> rcl:L-US0204/7
Changed lines of the file:
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@@
 <part name="L1" library="rcl" deviceset="L-US" device="6000-XXX-RC" value="210uH"/>
 <part name="GND20" library="supply1" deviceset="GND" device=""/>
-<part name="L2" library="rcl" deviceset="L-US" device="6000-XXX-RC" value="1uH"/>
+<part name="L2" library="rcl" deviceset="L-US" device="0204/7" value="1uH"/>
 <part name="C5" library="rcl" deviceset="CPOL-EU" device="E2-5" value="100uF"/>
 <part name="GND21" library="supply1" deviceset="GND" device=""/>

Commit message: Ajustes
Parts:
- C2, C4: device rcl:CPOL-EUE2.5-7 -> rcl:CPOL-EUE3.5-8
- C5: device rcl:CPOL-EUE2-5 -> rcl:CPOL-EUE3.5-8
Changed lines of the file:
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@@
 <part name="P+8" library="supply1" deviceset="VCC" device="" value="+8V"/>
 <part name="IC5" library="mc34063" deviceset="MC34063" device="AP"/>
-<part name="C2" library="rcl" deviceset="CPOL-EU" device="E2.5-7" value="100uF @ 35V"/>
+<part name="C2" library="rcl" deviceset="CPOL-EU" device="E3.5-8" value="100uF @ 35V"/>
 <part name="GND15" library="supply1" deviceset="GND" device=""/>
 <part name="R14" library="rcl" deviceset="R-EU_" device="0207/7" value="2.4k"/>
@@
 <part name="C3" library="rcl" deviceset="C-EU" device="025-025X050" value="200pF"/>
 <part name="GND19" library="supply1" deviceset="GND" device=""/>
-<part name="C4" library="rcl" deviceset="CPOL-EU" device="E2.5-7" value="25uF"/>
+<part name="C4" library="rcl" deviceset="CPOL-EU" device="E3.5-8" value="25uF"/>
 <part name="L1" library="rcl" deviceset="L-US" device="6000-XXX-RC" value="210uH"/>
 <part name="GND20" library="supply1" deviceset="GND" device=""/>
 <part name="L2" library="rcl" deviceset="L-US" device="0204/7" value="1uH"/>
-<part name="C5" library="rcl" deviceset="CPOL-EU" device="E2-5" value="100uF"/>
+<part name="C5" library="rcl" deviceset="CPOL-EU" device="E3.5-8" value="100uF"/>
 <part name="GND21" library="supply1" deviceset="GND" device=""/>
 <part name="P+9" library="supply1" deviceset="VCC" device="" value="+8V"/>
