File: IronDriverRevA/IronDriverRevA.brd (EAGLE design)
At the start: 100 x 60 mm, 34 parts, among them IC1 PIC18F2550, IC2 OPA2376, IC3 7805TV, IC5 LM334

Commit message: Routing IronDriver
Parts:
- removed C2, C5: 10uF, rcl:C0805
- removed C3, C4: (no value), rcl:C0805
- removed IC5: LM334, LM334:TO-92
- added IC4: TL072P, linear:DIL08
- added Q1: BC557C, transistor-pnp:TO92-EBC
- IC2: value OPA2376 -> TL074P; device OPA2376:MSOP-8 -> linear:DIL14
- R10: value 9k -> (none); device rcl:R0805 -> rcl:0207/7
- R11: device rcl:R0805 -> rcl:0207/7
- R7: value 3.1k -> (none); device rcl:R0805 -> rcl:0207/7
- R8: value 79.7k -> (none); device rcl:R0805 -> rcl:0207/7
- R9: value 1k -> (none); device rcl:R0805 -> rcl:0207/7
- moved IC2 75.4 mm to (42.9, -28.7), flipped to the top, turned to 270 degrees
- moved R7 67.6 mm to (56.2, -35.0), flipped to the top, turned to 90 degrees
- moved R10 55.3 mm to (53.1, -35.0), flipped to the top, turned to 270 degrees
- moved R8 51.6 mm to (42.8, -39.5), flipped to the top
- moved R9 44.2 mm to (42.9, -17.3), flipped to the top
- moved R11 25.5 mm to (20.0, -26.4), flipped to the top, turned to 180 degrees
- moved J1 3.70 mm to (92.3, 29.7)
- moved R6 1.36 mm to (65.5, 48.4), turned to 0 degrees
Connections:
- removed net BUFEFR_OUT: IC2.P$6, IC2.P$7
- removed net BUFFER_IN: C3.1, IC2.P$5, R11.2
- removed net N$13: C5.2, R7.2, R8.1
- removed net N$14: R7.1
- removed net N$15: IC5.P$3
- removed net N$7: PTC.3
- removed net VREF-: IC1.4
- new net +8V: IC2.4, IC4.8, R11.1
- new net +PTC: IC2.3, IC4.2, PTC.1, R11.2
- new net -PTC: IC2.5, PTC.2, Q1.E
- new net N$19: IC2.12, IC2.8, R7.2
- new net N$21: IC4.3
- new net VGND: IC1.4, IC4.6, IC4.7, R10.2
- net ADC_IN: now also IC2.13, IC2.14
- net GND: now also IC2.11, IC4.4, PTC.3, Q1.C; no longer C2.2, C3.2, C4.2, IC2.P$4, R9.1
- net N$12: now also IC2.6, IC2.7, R8.1; no longer C2.1, IC2.P$3, R8.2
- net N$2: now also IC4.1, Q1.B; no longer C5.1, IC2.P$1, R10.2, R11.1
- net N$5: now also IC2.9, R7.1, R8.2; no longer PTC.1
- net N$6: now also IC2.10, R10.1, R9.2; no longer PTC.2
- net N$9: now also IC2.1, IC2.2, R9.1; no longer IC2.P$2, R10.1, R9.2
- net VCC: no longer C4.1, IC2.P$8, IC5.P$1
Routing:
- net N$19: track 0.00 -> 37.4 mm
- net GND: track 43.9 -> 72.2 mm
- net N$6: track 0.00 -> 25.4 mm
- net LCD_RW: track 0.00 -> 24.6 mm
- net ENC_B: track 0.00 -> 22.2 mm
- net N$5: track 0.00 -> 21.6 mm
- net LCD_RS: track 0.00 -> 17.0 mm
- net PGC: track 0.00 -> 16.1 mm
- net ENC_A: track 0.00 -> 14.9 mm
- net PGD: track 0.00 -> 13.1 mm
- net VPP: track 0.00 -> 9.29 mm
- net N$9: track 0.00 -> 6.32 mm
- net N$12: track 0.00 -> 5.82 mm
- net VGND: track 0.00 -> 5.02 mm
- net ADC_IN: track 0.00 -> 2.54 mm
Other:
- board size 100 x 60 mm -> 100 x 100 mm

Commit message: Routing
Parts:
- added R12, R13: 10k, rcl:RTRIM3296W
- R10, R7, R8, R9: value (none) -> 100k
- R11: value (none) -> 220
- R3, R6: device rcl:R0805 -> rcl:0207/7
- moved Q1 112.4 mm to (42.4, 74.3)
- moved IC4 110.3 mm to (30.9, 74.1), turned to 180 degrees
- moved R7 106.5 mm to (58.1, 71.5)
- moved R11 102.2 mm to (37.8, 74.2), turned to 90 degrees
- moved IC2 101.8 mm to (50.5, 72.8)
- moved R10 101.8 mm to (60.7, 66.5)
- moved R8 101.8 mm to (50.4, 62.0)
- moved R9 101.0 mm to (50.5, 83.4)
- moved R5 22.8 mm to (48.3, 36.2)
- moved R6 3.93 mm to (65.0, 44.5), flipped to the top, turned to 270 degrees
- moved R3 3.87 mm to (48.3, 33.3), flipped to the top, turned to 0 degrees
- moved OPTO1 1.20 mm to (35.6, 22.6)
- moved MOC1 0.16 mm to (35.6, 38.8)
Connections:
- new net N$7: IC4.5, R13.2
- net +8V: now also R12.3, R13.3
- net GND: now also R12.1, R13.1
- net N$21: now also R12.2
Routing:
- net GND: track 72.2 -> 246.6 mm
- net +PTC: track 0.00 -> 73.8 mm
- net VGND: track 5.02 -> 78.1 mm
- net -PTC: track 0.00 -> 70.6 mm
- net ADC_IN: track 2.54 -> 53.0 mm
- net +8V: track 0.00 -> 36.2 mm
- net HEATER: track 0.00 -> 23.7 mm
- net N$19: track 37.4 -> 24.5 mm
- net N$21: track 0.00 -> 9.80 mm
- net N$2: track 0.00 -> 9.40 mm
- net N$5: track 21.6 -> 12.9 mm
- net N$7: track 0.00 -> 6.70 mm
- net VPP: track 9.29 -> 14.6 mm
- net N$1: track 0.00 -> 5.07 mm
- net N$4: track 15.6 -> 14.2 mm
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
Commit message: Routing
Parts:
- moved C1 36.5 mm to (82.1, 63.5)
- moved IC1 36.5 mm to (75.0, 68.2)
- moved ICSP 36.5 mm to (75.1, 94.0)
- moved J1 36.5 mm to (93.2, 66.2)
- moved R6 36.5 mm to (65.9, 81.0)
- moved R12 14.5 mm to (35.5, 67.4), turned to 270 degrees
- moved Q1 13.5 mm to (35.6, 86.0), turned to 180 degrees
- moved R11 8.26 mm to (35.4, 82.1), turned to 180 degrees
- moved R13 6.02 mm to (35.5, 62.5)
- moved IC4 4.73 mm to (35.5, 75.2), turned to 270 degrees
- moved R4 1.10 mm to (16.7, 36.4)
Routing:
- net GND: track 246.6 -> 376.0 mm
- net -PTC: track 70.6 -> 118.3 mm
- net ADC_IN: track 53.0 -> 21.2 mm
- net VCC: track 0.00 -> 22.8 mm
- net VGND: track 78.1 -> 62.3 mm
- net HEATER: track 23.7 -> 35.3 mm
- net N$7: track 6.70 -> 14.7 mm
- net +8V: track 36.2 -> 29.4 mm
- net ZEROCROSSING: track 12.6 -> 17.3 mm
- net +PTC: track 73.8 -> 74.6 mm
- net N$6: track 24.5 -> 23.9 mm
- net N$10: track 15.1 -> 15.6 mm
- net N$21: track 9.80 -> 9.30 mm

Commit message: Routing
Parts:
- moved IC4 4.60 mm to (40.1, 75.3)
- moved Q1 4.60 mm to (40.2, 86.0)
- moved R11 4.60 mm to (40.0, 82.1)
- moved R12 4.60 mm to (40.1, 67.4)
- moved R13 4.60 mm to (40.1, 62.5)
- moved ICSP 3.90 mm to (75.0, 90.1)
- moved R6 3.18 mm to (68.1, 83.3)
- moved IC2 3.10 mm to (53.6, 72.8)
- moved R7 3.10 mm to (61.2, 71.5)
- moved R8 3.10 mm to (53.5, 62.0)
- moved R9 3.10 mm to (53.6, 83.4)
- moved R10 3.10 mm to (63.8, 66.5)
- moved C1 0.32 mm to (82.0, 63.2)
Routing:
- net LCD_E: track 0.00 -> 30.6 mm
- net LCD_RW: track 24.6 -> 41.3 mm
- net GND: track 376.0 -> 384.5 mm
- net -PTC: track 118.3 -> 126.6 mm
- net VGND: track 62.3 -> 55.0 mm
- net +PTC: track 74.6 -> 80.8 mm
- net VPP: track 14.6 -> 10.2 mm
- net PGD: track 13.1 -> 8.95 mm
- net ADC_IN: track 21.2 -> 18.1 mm
- net PGC: track 16.1 -> 13.8 mm
- net HEATER: track 35.3 -> 36.3 mm
- net ZEROCROSSING: track 17.3 -> 16.6 mm
- net VCC: track 22.8 -> 23.3 mm

Commit message: Routing
Parts:
- removed D1, D2, D3, D4: (no value), diode:DO41-10
- added C2: (no value), rcl:C0805
- added IC5: (no value), LM2596:TO-220
- added IC6: (no value), RS207:RS207
- moved PTC 29.3 mm to (29.9, 64.0)
- moved R10 5.05 mm to (63.1, 71.5), turned to 90 degrees
- moved Q1 1.75 mm to (42.0, 86.0)
- moved IC4 1.75 mm to (41.9, 75.3)
- moved R11 1.75 mm to (41.8, 82.1)
- moved R12 1.75 mm to (41.9, 67.4)
- moved R13 1.75 mm to (41.9, 62.5)
- moved R7 0.65 mm to (60.5, 71.5)
Connections:
- removed net N$16: D1.C, D4.C
- net +8V: now also C2.1
- net GND: now also C2.2, IC5.P$3, IC6.P$4; no longer D2.A, D3.A
- net LIVE: now also IC6.P$3; no longer D1.A, D3.C
- net NEUTRAL: now also IC6.P$2; no longer D2.C, D4.A
Routing:
- net GND: track 384.5 -> 323.1 mm
- net -PTC: track 126.6 -> 74.2 mm
- net +PTC: track 80.8 -> 45.6 mm
- net LIVE: track 39.2 -> 47.3 mm
- net NEUTRAL: track 40.8 -> 48.1 mm
- net HEATER: track 36.3 -> 40.2 mm
- net N$16: track 3.00 -> 0.00 mm
- net LCD_RW: track 41.3 -> 43.8 mm
- net VGND: track 55.0 -> 57.2 mm
- net N$2: track 9.82 -> 11.4 mm
- net N$6: track 23.9 -> 25.2 mm
- net LCD_E: track 30.6 -> 31.8 mm
- net N$21: track 9.40 -> 8.17 mm
- net +8V: track 29.6 -> 28.9 mm
- net N$5: track 12.8 -> 12.1 mm

Commit message: Added ChikenControlelr
Parts:
- added JUMPER1: (no value), rcl:M1206
Changed lines of the file:
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@@
 <element name="IC6" library="RS207" package="RS207" value="" x="35.6" y="9.2" rot="R90"/>
 <element name="C2" library="rcl" package="C0805" value="" x="41.4" y="75.05" rot="MR0"/>
+<element name="JUMPER1" library="rcl" package="M1206" value="" x="-15.05" y="70.45" rot="MR270"/>
 </elements>
 <signals>
